File: cp_midi_control_surface_002.kicad_pcb (KiCad board)
At the start: 2 copper layers, 101.6 x 53.3 mm, 13 parts, among them P1 Digital, P10 CONN_01X01, P11 CONN_01X01, P12 CONN_01X01, P13 CONN_01X01, P2 Power, P3 Analog, P4 Analog, P5 PWM, P6 PWM, P7 Communication, P8 CONN_01X01, P9 CONN_01X01

Commit message: Transfer of schematic from 002.0
Parts:
- added D1: ~, cunabulapress-footprints:LED_D3.0mm_EDIT, F.Cu at (467.6, 130.4)
- added D10: ~, cunabulapress-footprints:LED_D3.0mm_EDIT, F.Cu at (482.3, 130.4)
- added D11: ~, cunabulapress-footprints:LED_D3.0mm_EDIT, F.Cu at (477.4, 139.5)
- added D12: ~, cunabulapress-footprints:LED_D3.0mm_EDIT, F.Cu at (482.3, 135.0)
- added D13: ~, cunabulapress-footprints:LED_D3.0mm_EDIT, F.Cu at (487.2, 130.4)
- added D14: ~, cunabulapress-footprints:LED_D3.0mm_EDIT, F.Cu at (482.3, 139.5)
- added D15: ~, cunabulapress-footprints:LED_D3.0mm_EDIT, F.Cu at (462.7, 135.0)
- added D16: ~, cunabulapress-footprints:LED_D3.0mm_EDIT, F.Cu at (472.5, 139.5)
- added D2: ~, cunabulapress-footprints:LED_D3.0mm_EDIT, F.Cu at (462.7, 130.4)
- added D3: ~, cunabulapress-footprints:LED_D3.0mm_EDIT, F.Cu at (462.7, 139.5)
- added D4: ~, cunabulapress-footprints:LED_D3.0mm_EDIT, F.Cu at (467.6, 135.0)
- added D5: ~, cunabulapress-footprints:LED_D3.0mm_EDIT, F.Cu at (472.5, 130.4)
- added D6: ~, cunabulapress-footprints:LED_D3.0mm_EDIT, F.Cu at (467.6, 139.5)
- added D7: ~, cunabulapress-footprints:LED_D3.0mm_EDIT, F.Cu at (472.5, 135.0)
- added D8: ~, cunabulapress-footprints:LED_D3.0mm_EDIT, F.Cu at (477.4, 130.4)
- added D9: ~, cunabulapress-footprints:LED_D3.0mm_EDIT, F.Cu at (477.4, 135.0)
- added H1: MountingHole, cunabulapress-footprints:Mounting_Hole_3.2mm_M3, F.Cu at (442.2, 149.2)
- added H10: MountingHole, cunabulapress-footprints:Mounting_Hole_3.2mm_M3, F.Cu at (438.9, 163.3)
- added H11: MountingHole, cunabulapress-footprints:Mounting_Hole_3.2mm_M3, F.Cu at (437.2, 169.5)
- added H12: MountingHole, cunabulapress-footprints:Mounting_Hole_3.2mm_M3, F.Cu at (448.3, 158.6)
- added H13: MountingHole, cunabulapress-footprints:Mounting_Hole_3.2mm_M3, F.Cu at (443.6, 163.3)
- added H14: MountingHole, cunabulapress-footprints:Mounting_Hole_3.2mm_M3, F.Cu at (432.5, 169.5)
- added H15: MountingHole, cunabulapress-footprints:Mounting_Hole_3.2mm_M3, F.Cu at (448.3, 163.3)
- added H16: MountingHole, cunabulapress-footprints:Mounting_Hole_3.2mm_M3, F.Cu at (453.0, 158.6)
- added H17: MountingHole, cunabulapress-footprints:Mounting_Hole_3.2mm_M3, F.Cu at (442.0, 172.8)
- added H18: MountingHole, cunabulapress-footprints:Mounting_Hole_3.2mm_M3, F.Cu at (446.9, 149.2)
- added H19: MountingHole, cunabulapress-footprints:Mounting_Hole_3.2mm_M3, F.Cu at (446.7, 168.1)
- added H2: MountingHole, cunabulapress-footprints:Mounting_Hole_3.2mm_M3, F.Cu at (437.5, 153.9)
- added H20: MountingHole, cunabulapress-footprints:Mounting_Hole_3.2mm_M3, F.Cu at (434.2, 164.8)
- added H21: MountingHole, cunabulapress-footprints:Mounting_Hole_3.2mm_M3, F.Cu at (438.9, 158.6)
- added H22: MountingHole, cunabulapress-footprints:Mounting_Hole_3.2mm_M3, F.Cu at (424.7, 160.1)
- added H23: MountingHole, cunabulapress-footprints:Mounting_Hole_3.2mm_M3, F.Cu at (429.4, 160.1)
- added H24: MountingHole, cunabulapress-footprints:Mounting_Hole_3.2mm_M3, F.Cu at (424.7, 164.8)
- added H25: MountingHole, cunabulapress-footprints:Mounting_Hole_3.2mm_M3, F.Cu at (429.4, 164.8)
- added H26: MountingHole, cunabulapress-footprints:Mounting_Hole_3.2mm_M3, F.Cu at (434.2, 160.1)
- added H3: MountingHole, cunabulapress-footprints:Mounting_Hole_3.2mm_M3, F.Cu at (437.5, 149.2)
- added H4: MountingHole, cunabulapress-footprints:Mounting_Hole_3.2mm_M3, F.Cu at (442.0, 168.1)
- added H5: MountingHole, cunabulapress-footprints:Mounting_Hole_3.2mm_M3, F.Cu at (442.2, 153.9)
- added H6: MountingHole, cunabulapress-footprints:Mounting_Hole_3.2mm_M3, F.Cu at (446.9, 153.9)
- added H7: MountingHole, cunabulapress-footprints:Mounting_Hole_3.2mm_M3, F.Cu at (451.7, 149.2)
- added H8: MountingHole, cunabulapress-footprints:Mounting_Hole_3.2mm_M3, F.Cu at (451.7, 153.9)
- added H9: MountingHole, cunabulapress-footprints:Mounting_Hole_3.2mm_M3, F.Cu at (443.6, 158.6)
- added J1: Conn_01x08_Male, Connector_PinHeader_2.54mm:PinHeader_1x08_P2.54mm_Vertical, F.Cu at (257.8, -24.2)
- added J10: Conn_01x08_Female, cunabulapress-footprints:Connector_TE_Connectivity_Micro-MaTch_8_Position_Female, F.Cu at (415.2, 168.9)
- added J11: Conn_01x08_Female, cunabulapress-footprints:Connector_TE_Connectivity_Micro-MaTch_8_Position_Female, F.Cu at (428.0, 168.9)
- added J12: Conn_01x08_Female, cunabulapress-footprints:Connector_TE_Connectivity_Micro-MaTch_8_Position_Female, F.Cu at (433.0, 148.3)
- added J13: Conn_01x08_Female, cunabulapress-footprints:Connector_TE_Connectivity_Micro-MaTch_8_Position_Female, F.Cu at (433.0, 153.7)
- added J14: Conn_01x08_Female, cunabulapress-footprints:Connector_TE_Connectivity_Micro-MaTch_8_Position_Female, F.Cu at (523.2, 76.1)
- added J15: Conn_01x08_Female, cunabulapress-footprints:Connector_TE_Connectivity_Micro-MaTch_8_Position_Female, F.Cu at (442.2, 129.6)
- added J16: Conn_01x08_Female, cunabulapress-footprints:Connector_TE_Connectivity_Micro-MaTch_8_Position_Female, F.Cu at (564.6, 59.5)
- added J17: Conn_01x08_Female, cunabulapress-footprints:Connector_TE_Connectivity_Micro-MaTch_8_Position_Female, F.Cu at (470.9, 149.7)
- added J18: Conn_01x01_Male, cunabulapress-footprints:Arduino_1pin_EDIT, F.Cu at (406.3, 174.5)
- added J19: Conn_01x01_Male, cunabulapress-footprints:Arduino_1pin_EDIT, F.Cu at (409.6, 174.5)
- added J2: Conn_01x08_Male, Connector_PinHeader_2.54mm:PinHeader_1x08_P2.54mm_Vertical, F.Cu at (246.9, -24.2)
- added J20: Conn_01x01_Male, cunabulapress-footprints:Arduino_1pin_EDIT, F.Cu at (412.9, 174.5)
- added J21: Conn_01x01_Male, cunabulapress-footprints:Arduino_1pin_EDIT, F.Cu at (416.2, 174.5)
- added J22: Conn_01x01_Male, cunabulapress-footprints:Arduino_1pin_EDIT, F.Cu at (419.5, 174.5)
- added J23: Conn_01x01_Male, cunabulapress-footprints:Arduino_1pin_EDIT, F.Cu at (422.8, 174.5)
- added J3: Conn_01x08_Male, Connector_PinHeader_2.54mm:PinHeader_1x08_P2.54mm_Vertical, F.Cu at (171.8, 5.99)
- added J4: Conn_01x01_Male, Connector_PinHeader_2.54mm:PinHeader_1x01_P2.54mm_Vertical, F.Cu at (175.5, 5.99)
- added J5: Conn_01x01_Male, Connector_PinHeader_2.54mm:PinHeader_1x01_P2.54mm_Vertical, F.Cu at (179.1, 5.99)
- added J6: Conn_01x01_Male, Connector_PinHeader_2.54mm:PinHeader_1x01_P2.54mm_Vertical, F.Cu at (182.8, 5.99)
- added J7: Conn_01x01_Male, Connector_PinHeader_2.54mm:PinHeader_1x01_P2.54mm_Vertical, F.Cu at (186.4, 5.99)
- added J8: Conn_01x08_Male, Connector_PinHeader_2.54mm:PinHeader_1x08_P2.54mm_Vertical, F.Cu at (250.5, -24.2)
- added J9: Conn_01x08_Male, Connector_PinHeader_2.54mm:PinHeader_1x08_P2.54mm_Vertical, F.Cu at (254.2, -24.2)
- added PT_1: 10k, cunabulapress-footprints:Potentiometer_Alps_RK09K_Single_Vertical_Edit, F.Cu at (461.9, 68.1)
- added PT_10: 10k, cunabulapress-footprints:Potentiometer_Alps_RK09K_Single_Vertical_Edit, F.Cu at (461.9, 118.2)
- added PT_11: 10k, cunabulapress-footprints:Potentiometer_Alps_RK09K_Single_Vertical_Edit, F.Cu at (482.2, 101.5)
- added PT_12: 10k, cunabulapress-footprints:Potentiometer_Alps_RK09K_Single_Vertical_Edit, F.Cu at (502.4, 84.8)
- added PT_13: 10k, cunabulapress-footprints:Potentiometer_Alps_RK09K_Single_Vertical_Edit, F.Cu at (522.7, 68.1)
- added PT_14: 10k, cunabulapress-footprints:Potentiometer_Alps_RK09K_Single_Vertical_Edit, F.Cu at (482.2, 118.2)
- added PT_15: 10k, cunabulapress-footprints:Potentiometer_Alps_RK09K_Single_Vertical_Edit, F.Cu at (441.7, 68.1)
- added PT_16: 10k, cunabulapress-footprints:Potentiometer_Alps_RK09K_Single_Vertical_Edit, F.Cu at (441.7, 84.8)
- added PT_17: 10k, cunabulapress-footprints:Potentiometer_Alps_RK09K_Single_Vertical_Edit, F.Cu at (367.9, 156.9)
- added PT_18: 10k, cunabulapress-footprints:Potentiometer_Alps_RK09K_Single_Vertical_Edit, F.Cu at (306.4, 206.5)
- added PT_19: 10k, cunabulapress-footprints:Potentiometer_Alps_RK09K_Single_Vertical_Edit, F.Cu at (346.9, 173.6)
- added PT_2: 10k, cunabulapress-footprints:Potentiometer_Alps_RK09K_Single_Vertical_Edit, F.Cu at (441.7, 101.5)
- added PT_20: 10k, cunabulapress-footprints:Potentiometer_Alps_RK09K_Single_Vertical_Edit, F.Cu at (326.6, 190.3)
- added PT_21: 10k, cunabulapress-footprints:Potentiometer_Alps_RK09K_Single_Vertical_Edit, F.Cu at (367.1, 173.6)
- added PT_22: 10k, cunabulapress-footprints:Potentiometer_Alps_RK09K_Single_Vertical_Edit, F.Cu at (346.9, 190.3)
- added PT_23: 10k, cunabulapress-footprints:Potentiometer_Alps_RK09K_Single_Vertical_Edit, F.Cu at (326.6, 207.0)
- added PT_24: 10k, cunabulapress-footprints:Potentiometer_Alps_RK09K_Single_Vertical_Edit, F.Cu at (286.1, 206.5)
- added PT_25: 10k, cunabulapress-footprints:Potentiometer_Alps_RK09K_Single_Vertical_Edit, F.Cu at (388.1, 156.9)
- added PT_26: 10k, cunabulapress-footprints:Potentiometer_Alps_RK09K_Single_Vertical_Edit, F.Cu at (306.4, 189.8)
- added PT_27: 10k, cunabulapress-footprints:Potentiometer_Alps_RK09K_Single_Vertical_Edit, F.Cu at (326.6, 173.6)
- added PT_28: 10k, cunabulapress-footprints:Potentiometer_Alps_RK09K_Single_Vertical_Edit, F.Cu at (286.1, 189.8)
- added PT_29: 10k, cunabulapress-footprints:Potentiometer_Alps_RK09K_Single_Vertical_Edit, F.Cu at (286.1, 173.1)
- added PT_3: 10k, cunabulapress-footprints:Potentiometer_Alps_RK09K_Single_Vertical_Edit, F.Cu at (502.4, 101.5)
- added PT_30: 10k, cunabulapress-footprints:Potentiometer_Alps_RK09K_Single_Vertical_Edit, F.Cu at (306.4, 173.1)
- added PT_31: 10k, cunabulapress-footprints:Potentiometer_Alps_RK09K_Single_Vertical_Edit, F.Cu at (347.6, 156.9)
- added PT_4: 10k, cunabulapress-footprints:Potentiometer_Alps_RK09K_Single_Vertical_Edit, F.Cu at (461.9, 84.8)
- added PT_5: 10k, cunabulapress-footprints:Potentiometer_Alps_RK09K_Single_Vertical_Edit, F.Cu at (482.2, 68.1)
- added PT_6: 10k, cunabulapress-footprints:Potentiometer_Alps_RK09K_Single_Vertical_Edit, F.Cu at (441.7, 118.2)
- added PT_7: 10k, cunabulapress-footprints:Potentiometer_Alps_RK09K_Single_Vertical_Edit, F.Cu at (461.9, 101.5)
- added PT_8: 10k, cunabulapress-footprints:Potentiometer_Alps_RK09K_Single_Vertical_Edit, F.Cu at (482.2, 84.8)
- added PT_9: 10k, cunabulapress-footprints:Potentiometer_Alps_RK09K_Single_Vertical_Edit, F.Cu at (502.4, 68.1)
- added RN1: R_Network09, Resistor_THT:R_Array_SIP10, F.Cu at (171.7, -24.3)
- added RN2: R_Network08, Resistor_THT:R_Array_SIP9, F.Cu at (223.0, -24.3)
- added RN3: R_Network08, Resistor_THT:R_Array_SIP9, F.Cu at (223.0, -21.0)
- added RV1: 10k, cunabulapress-footprints:Potentiometer_Bourns_PTA4543_Single_Slide_CP_EDIT, F.Cu at (306.9, 66.1)
- added RV2: 10k, cunabulapress-footprints:Potentiometer_Bourns_PTA4543_Single_Slide_CP_EDIT, F.Cu at (306.9, 82.2)
- added RV3: 10k, cunabulapress-footprints:Potentiometer_Bourns_PTA4543_Single_Slide_CP_EDIT, F.Cu at (368.5, 66.1)
- added RV4: 10k, cunabulapress-footprints:Potentiometer_Bourns_PTA4543_Single_Slide_CP_EDIT, F.Cu at (306.9, 98.4)
- added RV5: 10k, cunabulapress-footprints:Potentiometer_Bourns_PTA4543_Single_Slide_CP_EDIT, F.Cu at (368.5, 82.2)
- added RV6: 10k, cunabulapress-footprints:Potentiometer_Bourns_PTA4543_Single_Slide_CP_EDIT, F.Cu at (306.9, 114.5)
- added RV7: 10k, cunabulapress-footprints:Potentiometer_Bourns_PTA4543_Single_Slide_CP_EDIT, F.Cu at (306.9, 130.7)
- added RV8: 10k, cunabulapress-footprints:Potentiometer_Bourns_PTA4543_Single_Slide_CP_EDIT, F.Cu at (368.5, 98.4)
- added RVCF1: R_POT, cunabulapress-footprints:Potentiometer_Bourns_PTA4543_Single_Slide_CP_EDIT, F.Cu at (306.9, 154.9)
- added RVM1: 10k, cunabulapress-footprints:Potentiometer_Bourns_PTA4543_Single_Slide_CP_EDIT, F.Cu at (368.5, 114.5)
- added SW1: SW_SPST_4_PIN, cunabulapress-footprints:Omron_B3F-5050, F.Cu at (346.4, -45.8)
- added SW10: SW_SPST_4_PIN, cunabulapress-footprints:Omron_B3F-5050, F.Cu at (376.2, -45.8)
- added SW11: SW_SPST_4_PIN, cunabulapress-footprints:Omron_B3F-5050, F.Cu at (361.4, -33.6)
- added SW12: SW_SPST_4_PIN, cunabulapress-footprints:Omron_B3F-5050, F.Cu at (346.4, -21.5)
- added SW13: SW_SPST_4_PIN, cunabulapress-footprints:Omron_B3F-5050, F.Cu at (376.2, -57.9)
- added SW14: SW_SPST_4_PIN, cunabulapress-footprints:Omron_B3F-5050, F.Cu at (361.4, -45.8)
- added SW15: SW_SPST_4_PIN, cunabulapress-footprints:Omron_B3F-5050, F.Cu at (346.4, -33.6)
- added SW16: SW_SPST_4_PIN, cunabulapress-footprints:Omron_B3F-5050, F.Cu at (361.4, -57.9)
- added SW17: SW_SPST_4_PIN, cunabulapress-footprints:Omron_B3F-5050, F.Cu at (376.2, 30.4)
- added SW18: SW_SPST_4_PIN, cunabulapress-footprints:Omron_B3F-5050, F.Cu at (406.1, -6.08)
- added SW19: SW_SPST_4_PIN, cunabulapress-footprints:Omron_B3F-5050, F.Cu at (391.1, 6.07)
- added SW2: SW_SPST_4_PIN, cunabulapress-footprints:Omron_B3F-5050, F.Cu at (346.4, -57.9)
- added SW20: SW_SPST_4_PIN, cunabulapress-footprints:Omron_B3F-5050, F.Cu at (376.2, 18.2)
- added SW21: SW_SPST_4_PIN, cunabulapress-footprints:Omron_B3F-5050, F.Cu at (361.4, 30.4)
- added SW22: SW_SPST_4_PIN, cunabulapress-footprints:Omron_B3F-5050, F.Cu at (391.1, -6.08)
- added SW23: SW_SPST_4_PIN, cunabulapress-footprints:Omron_B3F-5050, F.Cu at (376.2, 6.07)
- added SW24: SW_SPST_4_PIN, cunabulapress-footprints:Omron_B3F-5050, F.Cu at (391.1, 18.2)
- added SW25: SW_SPST_4_PIN, cunabulapress-footprints:Omron_B3F-5050, F.Cu at (361.4, 18.2)
- added SW26: SW_SPST_4_PIN, cunabulapress-footprints:Omron_B3F-5050, F.Cu at (346.4, 30.4)
- added SW27: SW_SPST_4_PIN, cunabulapress-footprints:Omron_B3F-5050, F.Cu at (376.2, -6.08)
- added SW28: SW_SPST_4_PIN, cunabulapress-footprints:Omron_B3F-5050, F.Cu at (361.4, 6.07)
- added SW29: SW_SPST_4_PIN, cunabulapress-footprints:Omron_B3F-5050, F.Cu at (346.4, 18.2)
- added SW3: SW_SPST_4_PIN, cunabulapress-footprints:Omron_B3F-5050, F.Cu at (391.1, -33.6)
- added SW30: SW_SPST_4_PIN, cunabulapress-footprints:Omron_B3F-5050, F.Cu at (361.4, -6.08)
- added SW31: SW_SPST_4_PIN, cunabulapress-footprints:Omron_B3F-5050, F.Cu at (346.4, 6.07)
- added SW32: SW_SPST_4_PIN, cunabulapress-footprints:Omron_B3F-5050, F.Cu at (346.4, -6.08)
- added SW33: SW_SPST_4_PIN, cunabulapress-footprints:Omron_B3F-5050, F.Cu at (481.0, 6.07)
- added SW34: SW_SPST_4_PIN, cunabulapress-footprints:Omron_B3F-5050, F.Cu at (481.0, -6.08)
- added SW35: SW_SPST_4_PIN, cunabulapress-footprints:Omron_B3F-5050, F.Cu at (466.1, 6.07)
- added SW36: SW_SPST_4_PIN, cunabulapress-footprints:Omron_B3F-5050, F.Cu at (466.1, -6.08)
- added SW37: SW_SPST_4_PIN, cunabulapress-footprints:Omron_B3F-5050, F.Cu at (436.3, -6.08)
- added SW38: SW_SPST_4_PIN, cunabulapress-footprints:Omron_B3F-5050, F.Cu at (451.2, 6.07)
- added SW39: SW_SPST_4_PIN, cunabulapress-footprints:Omron_B3F-5050, F.Cu at (451.2, -6.08)
- added SW4: SW_SPST_4_PIN, cunabulapress-footprints:Omron_B3F-5050, F.Cu at (376.2, -21.5)
- added SW40: SW_SPST_4_PIN, cunabulapress-footprints:Omron_B3F-5050, F.Cu at (436.3, 6.07)
- added SW41: SW_SPST_4_PIN, cunabulapress-footprints:Omron_B3F-5050, F.Cu at (481.0, -33.6)
- added SW42: SW_SPST_4_PIN, cunabulapress-footprints:Omron_B3F-5050, F.Cu at (466.1, -21.5)
- added SW43: SW_SPST_4_PIN, cunabulapress-footprints:Omron_B3F-5050, F.Cu at (495.9, -57.9)
- added SW44: SW_SPST_4_PIN, cunabulapress-footprints:Omron_B3F-5050, F.Cu at (481.0, -45.8)
- added SW45: SW_SPST_4_PIN, cunabulapress-footprints:Omron_B3F-5050, F.Cu at (466.1, -33.6)
- added SW46: SW_SPST_4_PIN, cunabulapress-footprints:Omron_B3F-5050, F.Cu at (451.2, -21.5)
- added SW47: SW_SPST_4_PIN, cunabulapress-footprints:Omron_B3F-5050, F.Cu at (481.0, -57.9)
- added SW48: SW_SPST_4_PIN, cunabulapress-footprints:Omron_B3F-5050, F.Cu at (466.1, -45.8)
- added SW49: SW_SPST_4_PIN, cunabulapress-footprints:Omron_B3F-5050, F.Cu at (451.2, -33.6)
- added SW5: SW_SPST_4_PIN, cunabulapress-footprints:Omron_B3F-5050, F.Cu at (406.1, -57.9)
- added SW50: SW_SPST_4_PIN, cunabulapress-footprints:Omron_B3F-5050, F.Cu at (436.3, -21.5)
- added SW51: SW_SPST_4_PIN, cunabulapress-footprints:Omron_B3F-5050, F.Cu at (466.1, -57.9)
- added SW52: SW_SPST_4_PIN, cunabulapress-footprints:Omron_B3F-5050, F.Cu at (451.2, -45.8)
- added SW53: SW_SPST_4_PIN, cunabulapress-footprints:Omron_B3F-5050, F.Cu at (436.3, -33.6)
- added SW54: SW_SPST_4_PIN, cunabulapress-footprints:Omron_B3F-5050, F.Cu at (451.2, -57.9)
- added SW55: SW_SPST_4_PIN, cunabulapress-footprints:Omron_B3F-5050, F.Cu at (436.3, -45.8)
- added SW56: SW_SPST_4_PIN, cunabulapress-footprints:Omron_B3F-5050, F.Cu at (436.3, -57.9)
- added SW6: SW_SPST_4_PIN, cunabulapress-footprints:Omron_B3F-5050, F.Cu at (391.1, -45.8)
- added SW7: SW_SPST_4_PIN, cunabulapress-footprints:Omron_B3F-5050, F.Cu at (376.2, -33.6)
- added SW8: SW_SPST_4_PIN, cunabulapress-footprints:Omron_B3F-5050, F.Cu at (361.4, -21.5)
- added SW9: SW_SPST_4_PIN, cunabulapress-footprints:Omron_B3F-5050, F.Cu at (391.1, -57.9)
- added SW_F1: SW_DIP_x10, Package_DIP:DIP-20_W7.62mm, F.Cu at (197.4, -24.4)
- added SW_M1: Mode Switch, cunabulapress-footprints:RotaryEncoder_Alps_EC12E_Vertical_H20mm_6_Preset_Silk_EDIT, F.Cu at (411.3, 157.9)
- added U1: CD74HC4067M, Package_SO:SOIC-24W_7.5x15.4mm_P1.27mm, F.Cu at (218.7, 12.2)
- added U2: CD74HC4067M, Package_SO:SOIC-24W_7.5x15.4mm_P1.27mm, F.Cu at (268.8, -17.9)
- added U3: CD74HC4067M, Package_SO:SOIC-24W_7.5x15.4mm_P1.27mm, F.Cu at (176.0, 37.6)
- added U4: CD74HC4067M, Package_SO:SOIC-24W_7.5x15.4mm_P1.27mm, F.Cu at (218.7, 32.0)
- added U5: CD74HC4067M, Package_SO:SOIC-24W_7.5x15.4mm_P1.27mm, F.Cu at (251.6, 6.78)
- P1: footprint Socket_Arduino_Mega:Socket_Strip_Arduino_2x18 -> Connector_PinSocket_2.54mm:PinSocket_1x18_P2.54mm_Vertical
- P3, P4: value Analog -> Analogue
- turned P1 to 180 degrees
Connections:
- net +3V3 renamed Net-(P2-Pad4)
- net /0(Rx0) renamed Net-(P6-Pad8)
- net /1(Tx0) renamed Net-(P6-Pad7)
- net /41 renamed Net-(P1-Pad16)
- net /A12 renamed Net-(P4-Pad5)
- net /A13 renamed Net-(P4-Pad6)
- net /A14 renamed Net-(P4-Pad7)
- net /A15 renamed Net-(P4-Pad8)
- net /AREF renamed Net-(P5-Pad3)
- net /IOREF renamed Net-(P2-Pad2)
- net /Reset renamed Net-(P2-Pad3)
- net /SCL renamed Net-(P5-Pad1)
- net /SDA renamed Net-(P5-Pad2)
- net /Vin renamed Net-(P2-Pad8)
- P1 pad 10: /47 -> /36
- P1 pad 11: /44 -> /34
- P1 pad 12: /45 -> /32
- P1 pad 13: /42 -> Net-(P1-Pad13)
- P1 pad 14: /43 -> /28
- P1 pad 15: /40 -> /26
- P1 pad 17: /38 -> Net-(P1-Pad17)
- P1 pad 18: /39 -> +5V
- P1 pad 2: GND -> /52
- P1 pad 3: /52(SCK) -> /50
- P1 pad 4: /53(SS) -> /48
- P1 pad 5: /50(MISO) -> /46
- P1 pad 6: /51(MOSI) -> /44
- P1 pad 7: /48 -> /42
- P1 pad 8: /49 -> /40
- P1 pad 9: /46 -> /38
- P2 pad 7: GND -> Net-(P2-Pad7)
- P5 pad 10: /8(**) -> /8
- P5 pad 5: /13(**) -> /13
- P5 pad 6: /12(**) -> /12
- P5 pad 7: /11(**) -> /11
- P5 pad 8: /10(**) -> /10
- P5 pad 9: /9(**) -> /9
- P6 pad 1: /7(**) -> /7
- P6 pad 2: /6(**) -> /6
- P6 pad 3: /5(**) -> /5
- P6 pad 4: /4(**) -> /4
- P6 pad 5: /3(**) -> /3
- P6 pad 6: /2(**) -> /2
- P7 pad 1: /14(Tx3) -> /14
- P7 pad 2: /15(Rx3) -> /15
- P7 pad 3: /16(Tx2) -> /16
- P7 pad 4: /17(Rx2) -> /17
- P7 pad 5: /18(Tx1) -> Mult_4
- P7 pad 6: /19(Rx1) -> Mult_3
- P7 pad 7: /20(SDA) -> Mult_2
- P7 pad 8: /21(SCL) -> Mult_1
