File: cp_midi_control_surface_002.kicad_pcb (KiCad board)
At the start: 2 copper layers, 101.6 x 53.3 mm, 185 parts, among them J1 Conn_01x08_Male, J10 Conn_01x08_Female, J11 Conn_01x08_Female, J12 Conn_01x08_Female, J13 Conn_01x08_Female, J14 Conn_01x08_Female, J15 Conn_01x08_Female, J16 Conn_01x08_Female, J17 Conn_01x08_Female, J18 Conn_01x01_Male, J19 Conn_01x01_Male, J2 Conn_01x08_Male, J20 Conn_01x01_Male, J21 Conn_01x01_Male, J22 Conn_01x01_Male, J23 Conn_01x01_Male, J3 Conn_01x08_Male, J4 Conn_01x01_Male, J5 Conn_01x01_Male, J6 Conn_01x01_Male, J7 Conn_01x01_Male, J8 Conn_01x08_Male, J9 Conn_01x08_Male, P1 Digital, P10 CONN_01X01, P11 CONN_01X01, P12 CONN_01X01, P13 CONN_01X01, P2 Power, P3 Analogue, P4 Analogue, P5 PWM, P6 PWM, P7 Communication, P8 CONN_01X01, P9 CONN_01X01, SW1 SW_SPST_4_PIN, SW10 SW_SPST_4_PIN, SW11 SW_SPST_4_PIN, SW12 SW_SPST_4_PIN, SW13 SW_SPST_4_PIN, SW14 SW_SPST_4_PIN, SW15 SW_SPST_4_PIN, SW16 SW_SPST_4_PIN, SW17 SW_SPST_4_PIN, SW18 SW_SPST_4_PIN, SW19 SW_SPST_4_PIN, SW2 SW_SPST_4_PIN, SW20 SW_SPST_4_PIN, SW21 SW_SPST_4_PIN, SW22 SW_SPST_4_PIN, SW23 SW_SPST_4_PIN, SW24 SW_SPST_4_PIN, SW25 SW_SPST_4_PIN, SW26 SW_SPST_4_PIN, SW27 SW_SPST_4_PIN, SW28 SW_SPST_4_PIN, SW29 SW_SPST_4_PIN, SW3 SW_SPST_4_PIN, SW30 SW_SPST_4_PIN, SW31 SW_SPST_4_PIN, SW32 SW_SPST_4_PIN, SW33 SW_SPST_4_PIN, SW34 SW_SPST_4_PIN, SW35 SW_SPST_4_PIN, SW36 SW_SPST_4_PIN, SW37 SW_SPST_4_PIN, SW38 SW_SPST_4_PIN, SW39 SW_SPST_4_PIN, SW4 SW_SPST_4_PIN, SW40 SW_SPST_4_PIN, SW41 SW_SPST_4_PIN, SW42 SW_SPST_4_PIN, SW43 SW_SPST_4_PIN, SW44 SW_SPST_4_PIN, SW45 SW_SPST_4_PIN, SW46 SW_SPST_4_PIN, SW47 SW_SPST_4_PIN, SW48 SW_SPST_4_PIN, SW49 SW_SPST_4_PIN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

Commit message: Initial potentiometer layout
Parts:
- moved PT_13 376.7 mm to (189.0, 243.0)
- moved PT_9 346.6 mm to (189.0, 216.0)
- moved PT_5 317.1 mm to (189.0, 189.0)
- moved PT_14 294.0 mm to (216.0, 243.0)
- moved PT_1 288.6 mm to (189.0, 162.0)
- moved PT_25 278.1 mm to (189.0, 351.0)
- moved PT_12 266.9 mm to (270.0, 216.0)
- moved PT_3 266.4 mm to (243.0, 162.0)
- moved PT_11 265.2 mm to (243.0, 216.0)
- moved PT_15 264.7 mm to (243.0, 243.0)
- moved PT_10 264.7 mm to (216.0, 216.0)
- moved PT_6 236.5 mm to (216.0, 189.0)
- moved PT_8 236.4 mm to (270.0, 189.0)
- moved PT_7 235.8 mm to (243.0, 189.0)
- moved PT_2 233.6 mm to (216.0, 162.0)
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
Commit message: More initial layout
Parts:
- U4: moved to B.Cu
- moved SW33 572.5 mm to (-27.0, 270.0)
- moved SW34 554.6 mm to (0.00, 270.0)
- moved SW35 512.3 mm to (27.0, 270.0)
- moved SW13 503.2 mm to (-27.0, 243.0)
- moved SW9 499.9 mm to (-27.0, 216.0)
- moved SW5 498.5 mm to (-27.0, 189.0)
- moved SW36 496.0 mm to (54.0, 270.0)
- moved SW14 462.6 mm to (0.00, 243.0)
- moved SW10 458.4 mm to (0.00, 216.0)
- moved SW6 456.2 mm to (0.00, 189.0)
- moved SW37 449.9 mm to (81.0, 270.0)
- moved J2 448.2 mm to (650.9, 169.8)
- moved J4 448.2 mm to (579.5, 200.0)
- moved J5 448.2 mm to (583.1, 200.0)
- moved J6 448.2 mm to (586.8, 200.0)
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Other:
- outline, holes or cut-outs redrawn

Commit message: Further initial placement
Parts:
- U1, U2, U3, U5: moved to B.Cu
- moved U1 612.7 mm to (10.0, 203.8), turned to 270 degrees
- moved J15 566.0 mm to (14.2, 229.0)
- moved U2 553.9 mm to (119.5, 201.6), turned to 270 degrees
- moved U5 436.6 mm to (232.0, 306.5), turned to 90 degrees
- moved J14 400.6 mm to (230.5, 242.2)
- moved D16 390.6 mm to (189.0, 270.0), turned to 90 degrees
- moved D14 390.3 mm to (199.1, 270.0), turned to 90 degrees
- moved D13 390.0 mm to (204.2, 270.0), turned to 90 degrees
- moved D12 380.1 mm to (209.2, 270.0), turned to 90 degrees
- moved D15 375.7 mm to (194.1, 270.0), turned to 90 degrees
- moved D11 370.2 mm to (214.3, 270.0), turned to 90 degrees
- moved D10 370.0 mm to (219.4, 270.0), turned to 90 degrees
- moved D9 360.0 mm to (224.4, 270.0), turned to 90 degrees
- moved D8 354.9 mm to (229.5, 270.0), turned to 90 degrees
- moved U3 351.9 mm to (229.5, 200.0), turned to 270 degrees
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Routing:
- net +5V: track 0.00 -> 656.1 mm
- net Mult_1: track 0.00 -> 7.60 mm
- net Mult_3: track 0.00 -> 7.27 mm
- net Mult_2: track 0.00 -> 7.25 mm
- net Mult_4: track 0.00 -> 7.02 mm
- added copper zone on B.Cu, net GND
- added copper zone on F.Cu, net GND

Commit message: All panel components placed
Parts:
- J10, J12, J13, J14, J15, J16, J17, P1: moved to B.Cu
- P10, P11, P12, P13, P8, P9: footprint Socket_Arduino_Mega:Arduino_1pin -> cunabulapress-footprints:Mounting_Hole_M3_Target_Only
- P2, P3, P4, P6, P7: footprint Socket_Arduino_Mega:Socket_Strip_Arduino_1x08 -> Connector_PinHeader_2.54mm:PinHeader_1x08_P2.54mm_Vertical; moved to B.Cu
- P5: footprint Socket_Arduino_Mega:Socket_Strip_Arduino_1x10 -> Connector_PinHeader_2.54mm:PinHeader_1x10_P2.54mm_Vertical; moved to B.Cu
- moved J12 169.8 mm to (606.8, 253.5)
- moved SW13 111.0 mm to (78.8, 209.2)
- moved SW9 109.7 mm to (78.8, 186.8)
- moved RV1 109.1 mm to (78.8, 297.0)
- moved SW33 109.1 mm to (78.8, 243.0)
- moved SW5 108.6 mm to (78.8, 164.2)
- moved SW1 107.7 mm to (78.8, 141.8)
- moved SW14 106.7 mm to (101.2, 209.2)
- moved U1 106.3 mm to (112.5, 175.5)
- moved SW10 105.4 mm to (101.2, 186.8)
- moved RV2 104.8 mm to (101.2, 297.0)
- moved SW34 104.8 mm to (101.2, 243.0)
- moved SW6 104.2 mm to (101.2, 164.2)
- moved SW2 103.3 mm to (101.2, 141.8)
- moved SW15 102.5 mm to (123.8, 209.2)
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Routing:
- net Mult_1: track 7.60 -> 0.00 mm
- net Mult_3: track 7.27 -> 0.00 mm
- net Mult_2: track 7.25 -> 0.00 mm
- net Mult_4: track 7.02 -> 0.00 mm
- net +5V: track 656.1 -> 649.6 mm
Other:
- board outline removed

Commit message: Beginning button connections
Beginning running traces to the button blocks modified schematic to ensure minimum trace length, rotate buttons to achieve this.
Parts:
- moved SW48 67.5 mm to (384.8, 164.2), turned to 180 degrees
- moved SW8 67.5 mm to (78.8, 164.2), turned to 180 degrees
- moved SW1 50.3 mm to (123.8, 164.2), turned to 180 degrees
- moved SW2 50.3 mm to (146.2, 164.2), turned to 180 degrees
- moved SW41 50.3 mm to (429.8, 164.2), turned to 180 degrees
- moved SW42 50.3 mm to (452.2, 164.2), turned to 180 degrees
- moved SW45 31.8 mm to (407.2, 141.8), turned to 180 degrees
- moved SW46 31.8 mm to (384.8, 141.8), turned to 180 degrees
- moved SW5 31.8 mm to (101.2, 141.8), turned to 180 degrees
- moved SW6 31.8 mm to (78.8, 141.8), turned to 180 degrees
- moved SW3 22.5 mm to (146.2, 141.8), turned to 180 degrees
- moved SW4 22.5 mm to (123.8, 141.8), turned to 180 degrees
- moved SW43 22.5 mm to (452.2, 141.8), turned to 180 degrees
- moved SW44 22.5 mm to (429.8, 141.8), turned to 180 degrees
- moved SW47 22.5 mm to (407.2, 164.2), turned to 180 degrees
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Connections:
- U1 pad 2: Net-(SW8-Pad2) -> Net-(SW8-Pad1)
- U1 pad 3: Net-(SW7-Pad2) -> Net-(SW7-Pad1)
- U1 pad 4: Net-(SW6-Pad2) -> Net-(SW6-Pad1)
- U1 pad 5: Net-(SW5-Pad2) -> Net-(SW5-Pad1)
- U1 pad 6: Net-(SW4-Pad1) -> Net-(SW4-Pad2)
- U1 pad 7: Net-(SW3-Pad1) -> Net-(SW3-Pad2)
- U1 pad 8: Net-(SW2-Pad1) -> Net-(SW2-Pad2)
- U1 pad 9: Net-(SW1-Pad1) -> Net-(SW1-Pad2)
- U4 pad 2: Net-(SW48-Pad2) -> Net-(SW48-Pad1)
- U4 pad 4: Net-(SW46-Pad2) -> Net-(SW46-Pad1)
- U4 pad 5: Net-(SW45-Pad2) -> Net-(SW45-Pad1)
- U4 pad 6: Net-(SW44-Pad1) -> Net-(SW44-Pad2)
- U4 pad 7: Net-(SW43-Pad1) -> Net-(SW43-Pad2)
- U4 pad 8: Net-(SW42-Pad1) -> Net-(SW42-Pad2)
- U4 pad 9: Net-(SW41-Pad1) -> Net-(SW41-Pad2)
Routing:
- net +5V: track 649.6 -> 816.0 mm
- net Net-(SW43-Pad2): track 0.00 -> 45.1 mm
- net Net-(SW3-Pad2): track 0.00 -> 45.1 mm
- net Net-(SW6-Pad1): track 0.00 -> 42.6 mm
- net Net-(SW46-Pad1): track 0.00 -> 42.6 mm
- net Net-(SW42-Pad2): track 0.00 -> 31.8 mm
- net Net-(SW2-Pad2): track 0.00 -> 31.7 mm
- net Net-(SW4-Pad2): track 0.00 -> 28.9 mm
- net Net-(SW44-Pad2): track 0.00 -> 28.9 mm
- net Net-(SW45-Pad1): track 0.00 -> 27.8 mm
- net Net-(SW5-Pad1): track 0.00 -> 27.8 mm
- net Net-(SW49-Pad2): track 0.00 -> 26.0 mm
- net Net-(SW9-Pad2): track 0.00 -> 26.0 mm
- net Net-(SW48-Pad1): track 0.00 -> 25.9 mm
- net Net-(SW8-Pad1): track 0.00 -> 25.9 mm
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
Commit message: Further work on the separate boards
Parts:
- moved SW24 67.5 mm to (168.8, 164.2), turned to 180 degrees
- moved J17 62.7 mm to (474.8, 164.2)
- moved PT_1 60.4 mm to (324.0, 162.0)
- moved PT_11 60.4 mm to (270.0, 216.0)
- moved PT_12 60.4 mm to (297.0, 216.0)
- moved PT_2 60.4 mm to (351.0, 162.0)
- moved PT_13 54.0 mm to (324.0, 216.0)
- moved PT_14 54.0 mm to (351.0, 216.0)
- moved PT_7 54.0 mm to (270.0, 162.0)
- moved PT_8 54.0 mm to (297.0, 162.0)
- moved SW11 50.3 mm to (78.8, 209.2)
- moved SW12 50.3 mm to (101.2, 209.2)
- moved SW17 50.3 mm to (213.8, 164.2), turned to 180 degrees
- moved SW18 50.3 mm to (236.2, 164.2), turned to 180 degrees
- moved SW27 50.3 mm to (168.8, 209.2)
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Connections:
- U2 pad 2: Net-(SW24-Pad2) -> Net-(SW24-Pad1)
- U2 pad 4: Net-(SW22-Pad2) -> Net-(SW22-Pad1)
- U2 pad 5: Net-(SW21-Pad2) -> Net-(SW21-Pad1)
- U2 pad 6: Net-(SW20-Pad1) -> Net-(SW20-Pad2)
- U2 pad 7: Net-(SW19-Pad1) -> Net-(SW19-Pad2)
- U2 pad 8: Net-(SW18-Pad1) -> Net-(SW18-Pad2)
- U2 pad 9: Net-(SW17-Pad1) -> Net-(SW17-Pad2)
Routing:
- net +5V: track 816.0 -> 1397.3 mm
- net Net-(J17-Pad5): track 0.00 -> 138.8 mm
- net Net-(J15-Pad5): track 0.00 -> 136.6 mm
- net Net-(J16-Pad5): track 0.00 -> 134.7 mm
- net Net-(PT_3-Pad2): track 0.00 -> 65.0 mm
- net Net-(PT_6-Pad2): track 0.00 -> 62.5 mm
- net Net-(PT_14-Pad2): track 0.00 -> 61.9 mm
- net Net-(PT_11-Pad2): track 0.00 -> 60.8 mm
- net Net-(PT_2-Pad2): track 0.00 -> 54.3 mm
- net Net-(PT_7-Pad2): track 0.00 -> 52.4 mm
- net Net-(J15-Pad1): track 0.00 -> 48.9 mm
- net Net-(J16-Pad1): track 0.00 -> 46.9 mm
- net Net-(PT_4-Pad2): track 0.00 -> 46.9 mm
- net Net-(J15-Pad2): track 0.00 -> 46.1 mm
- net Net-(PT_5-Pad2): track 0.00 -> 45.8 mm
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
Commit message: Further connections
Parts:
- moved J13 159.3 mm to (423.8, 251.0)
- moved J15 81.0 mm to (146.2, 199.3)
- moved J14 33.0 mm to (341.7, 202.0)
- turned SW33 to 90 degrees
Routing:
- net Net-(J14-Pad5): track 0.00 -> 185.2 mm
- net Net-(J14-Pad1): track 0.00 -> 85.2 mm
- net Net-(J14-Pad2): track 0.00 -> 80.2 mm
- net Net-(J14-Pad3): track 0.00 -> 79.5 mm
- net Net-(J14-Pad4): track 0.00 -> 74.2 mm
- net +5V: track 1397.3 -> 1420.2 mm
- net Net-(J15-Pad3): track 38.3 -> 44.4 mm
- net Net-(J15-Pad1): track 48.9 -> 54.7 mm
- net Net-(J15-Pad2): track 46.1 -> 48.5 mm
- net Net-(PT_16-Pad2): track 13.7 -> 15.9 mm
- net Net-(PT_14-Pad2): track 61.9 -> 64.0 mm
- net Net-(PT_15-Pad2): track 42.6 -> 44.7 mm
- net Net-(J15-Pad4): track 36.6 -> 38.5 mm
- net Net-(J15-Pad5): track 136.6 -> 135.6 mm

Commit message: Connected Faders 1-8
Routing:
- net /A1: track 0.00 -> 367.8 mm
- net /A2: track 0.00 -> 342.2 mm
- net /A3: track 0.00 -> 316.7 mm
- net /A4: track 0.00 -> 291.1 mm
- net /A5: track 0.00 -> 265.6 mm
- net /A6: track 0.00 -> 240.1 mm
- net /A7: track 0.00 -> 214.5 mm
- net /A8: track 0.00 -> 186.5 mm
- net +5V: track 1420.2 -> 1386.4 mm
