File: cp_midi_control_surface_002.kicad_pcb (KiCad board)
At the start: 2 copper layers, 197 parts, among them P1 Power, P10 Guide, P11 Guide, P12 Guide, P13 Guide, P2 Analogue, P3 Digital, P4 Communication, P5 PWM, P6 PWM, P8 Guide, P9 Guide, SW1 B3F-5050, SW10 B3F-5050, SW11 B3F-5050, SW12 B3F-5050, SW13 B3F-5050, SW14 B3F-5050, SW15 B3F-5050, SW16 B3F-5050, SW17 B3F-5050, SW18 B3F-5050, SW19 B3F-5050, SW2 B3F-5050, SW20 B3F-5050, SW21 B3F-5050, SW22 B3F-5050, SW23 B3F-5050, SW24 B3F-5050, SW25 B3F-5050, SW26 B3F-5050, SW27 B3F-5050, SW28 B3F-5050, SW29 B3F-5050, SW3 B3F-5050, SW30 B3F-5050, SW31 B3F-5050, SW32 B3F-5050, SW33 B3F-5050, SW34 B3F-5050, SW35 B3F-5050, SW36 B3F-5050, SW37 B3F-5050, SW38 B3F-5050, SW39 B3F-5050, SW4 B3F-5050, SW40 B3F-5050, SW41 B3F-5050, SW42 B3F-5050, SW43 B3F-5050, SW44 B3F-5050, SW45 B3F-5050, SW46 B3F-5050, SW47 B3F-5050, SW48 B3F-5050, SW49 B3F-5050, SW5 B3F-5050, SW50 B3F-5050, SW51 B3F-5050, SW52 B3F-5050, SW53 B3F-5050, SW54 B3F-5050, SW55 B3F-5050, SW56 B3F-5050, SW6 B3F-5050, SW7 B3F-5050, SW8 B3F-5050, SW9 B3F-5050, U1 CD74HC4067M, U2 CD74HC4067M, U3 CD74HC4067M, U4 CD74HC4067M, U5 CD74HC4067M, U6 CD74HC4067M

Commit message: Further traces added and reassigned duaghter board connection
Connections:
- J10 pad 1: /53 -> /39
- J10 pad 2: /51 -> /41
- J10 pad 3: /49 -> /43
- J10 pad 4: /47 -> /45
- J12 pad 1: /45 -> /47
- J12 pad 2: /43 -> /49
- J12 pad 3: /41 -> /51
- J12 pad 4: /39 -> /53
- J2 pad 5: /A0 -> /A3
- J8 pad 5: /A3 -> /A0
Routing:
- net /47: track 0.00 -> 416.1 mm, vias 0 -> 2
- net /49: track 0.00 -> 394.7 mm, vias 0 -> 2
- net /51: track 0.00 -> 390.8 mm, vias 0 -> 2
- net /53: track 0.00 -> 387.0 mm, vias 0 -> 2
- net /13: track 0.00 -> 381.0 mm
- net /41: track 0.00 -> 374.1 mm, vias 0 -> 2
- net /12: track 0.00 -> 372.9 mm
- net /45: track 0.00 -> 370.1 mm, vias 0 -> 2
- net /39: track 0.00 -> 367.7 mm, vias 0 -> 2
- net /11: track 0.00 -> 364.8 mm
- net /10: track 0.00 -> 356.6 mm
- net /43: track 0.00 -> 354.9 mm, vias 0 -> 2
- net /9: track 0.00 -> 348.5 mm
- net /8: track 0.00 -> 340.2 mm
- net /7: track 0.00 -> 330.6 mm
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
Commit message: Connections complete
All traces mapped and DRC passed apart from interboard errors - should look into fixing those.
Connections:
- J2 pad 5: /A3 -> /A1
- J4 pad 5: /A1 -> /A3
- J6 pad 5: /A2 -> /A5
- U5 pad 1: /A5 -> /A2
- U6 pad 1: /Lower Pots/LOWER_POTS -> /A4
Routing:
- net Net-(RV3-Pad2): track 86.9 -> 480.2 mm
- net Net-(RV2-Pad2): track 56.4 -> 441.4 mm, vias 0 -> 1
- net Net-(RV8-Pad2): track 32.7 -> 400.4 mm, vias 0 -> 1
- net Net-(RV1-Pad2): track 32.4 -> 391.8 mm, vias 0 -> 1
- net /A1: track 0.00 -> 351.5 mm, vias 0 -> 2
- net Net-(RV7-Pad2): track 56.9 -> 393.5 mm, vias 0 -> 1
- net Net-(RV6-Pad2): track 81.1 -> 388.5 mm, vias 0 -> 1
- net /A2: track 0.00 -> 305.0 mm, vias 0 -> 2
- net Net-(RV5-Pad2): track 111.8 -> 389.5 mm, vias 0 -> 1
- net Net-(RV4-Pad2): track 136.5 -> 388.5 mm, vias 0 -> 1
- net /A3: track 0.00 -> 228.7 mm, vias 0 -> 2
- net /A4: track 0.00 -> 189.1 mm, vias 0 -> 2
- net Net-(RVM1-Pad2): track 205.0 -> 347.8 mm, vias 0 -> 2
- net /A5: track 2.96 -> 107.3 mm, vias 0 -> 1
- net +5V: track 2659.9 -> 2700.0 mm, vias 0 -> 1
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
Commit message: Cleaning up and rerouting traces
Connections:
- SW_F1 pad 1: Net-(RV1-Pad2) -> Net-(RV3-Pad2)
- SW_F1 pad 3: Net-(RV3-Pad2) -> Net-(RV1-Pad2)
- SW_F1 pad 4: Net-(RV4-Pad2) -> Net-(RV8-Pad2)
- SW_F1 pad 5: Net-(RV5-Pad2) -> Net-(RV7-Pad2)
- SW_F1 pad 7: Net-(RV7-Pad2) -> Net-(RV5-Pad2)
- SW_F1 pad 8: Net-(RV8-Pad2) -> Net-(RV4-Pad2)
Routing:
- net /13: track 381.0 -> 357.7 mm
- net /9: track 348.5 -> 325.3 mm
- net /12: track 372.9 -> 350.2 mm
- net /11: track 364.8 -> 342.2 mm
- net /8: track 340.2 -> 317.8 mm
- net /10: track 356.6 -> 334.7 mm
- net /7: track 330.6 -> 309.5 mm
- net Net-(RV4-Pad2): track 388.5 -> 408.6 mm
- net Net-(RV8-Pad2): track 400.4 -> 381.5 mm
- net /6: track 318.5 -> 301.3 mm
- net /5: track 267.5 -> 250.9 mm
- net /4: track 259.4 -> 243.4 mm
- net /3: track 251.2 -> 235.8 mm
- net Net-(RV5-Pad2): track 389.5 -> 404.8 mm
- net /2: track 243.1 -> 228.3 mm
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