File: _autosave-cp_midi_control_surface_002.kicad_pcb (KiCad board)
At the start: 2 copper layers, 421.6 x 332.7 mm, 174 parts, among them J1 Conn_02x05_Odd_Even, J2 Conn_02x05_Odd_Even, J7 Conn_02x05_Odd_Even, P1 Power, P11 Guide, P12 Guide, P13 Guide, P2 Analogue, P3 Digital, P4 Communication, P5 PWM, P6 PWM, P8 Guide, P9 Guide, SW1 B3F-5050, SW10 B3F-5050, SW11 B3F-5050, SW12 B3F-5050, SW13 B3F-5050, SW14 B3F-5050, SW15 B3F-5050, SW16 B3F-5050, SW17 B3F-5050, SW18 B3F-5050, SW19 B3F-5050, SW2 B3F-5050, SW20 B3F-5050, SW21 B3F-5050, SW22 B3F-5050, SW23 B3F-5050, SW24 B3F-5050, SW25 B3F-5050, SW26 B3F-5050, SW27 B3F-5050, SW28 B3F-5050, SW29 B3F-5050, SW3 B3F-5050, SW30 B3F-5050, SW31 B3F-5050, SW32 B3F-5050, SW4 B3F-5050, SW41 B3F-5050, SW42 B3F-5050, SW43 B3F-5050, SW44 B3F-5050, SW45 B3F-5050, SW46 B3F-5050, SW47 B3F-5050, SW48 B3F-5050, SW49 B3F-5050, SW5 B3F-5050, SW50 B3F-5050, SW51 B3F-5050, SW52 B3F-5050, SW53 B3F-5050, SW54 B3F-5050, SW55 B3F-5050, SW56 B3F-5050, SW6 B3F-5050, SW7 B3F-5050, SW8 B3F-5050, SW9 B3F-5050, U1 CD74HC4067M, U2 CD74HC4067M, U3 CD74HC4067M, U4 CD74HC4067M, U5 CD74HC4067M, U6 CD74HC4067M

Commit message: Added external connections / removed unused
+18 Buttons
+ Different connections for 7 spare multiplexer slots
- Unused Arduino pins
Parts:
- JA4: footprint Connector_PinHeader_2.54mm:PinHeader_2x05_P2.54mm_Vertical -> Connector_PinHeader_2.54mm:PinHeader_2x18_P2.54mm_Vertical
Connections:
- net Net-(J_EXT_1-Pad2) renamed /faders/U5_8
- net Net-(J_EXT_1-Pad3) renamed /faders/U5_9
- net Net-(J_EXT_1-Pad4) renamed /faders/U5_10
- net Net-(J_EXT_1-Pad5) renamed /faders/U5_11
- net Net-(J_EXT_1-Pad6) renamed /faders/U5_12
- net Net-(J_EXT_1-Pad7) renamed /faders/U5_13
- net Net-(J_EXT_1-Pad8) renamed /faders/U5_14
- JA4 pad 1: S0 -> Net-(JA4-Pad1)
- JA4 pad 2: S1 -> Net-(JA4-Pad2)
- JA4 pad 3: S2 -> Net-(JA4-Pad3)
- JA4 pad 4: S3 -> Net-(JA4-Pad4)
Routing:
- net /24: track 0.00 -> 185.6 mm
- net /22: track 0.00 -> 177.1 mm
