File: faders.sch (KiCad schematic (older format))
At the start: 13 parts, among them U5 CD74HC4067M

Commit message: Nearly there. Switch placed
Connections:
- net U5_10: now also U5.18 (I13); no longer U5.21 (I10)
- net U5_11: now also U5.19 (I12); no longer U5.20 (I11)
- net U5_12: now also U5.20 (I11); no longer U5.19 (I12)
- net U5_13: now also U5.21 (I10); no longer U5.18 (I13)
- net U5_14: now also U5.22 (I9); no longer U5.17 (I14)
- net U5_8: now also U5.16 (I15); no longer U5.23 (I8)
- net U5_9: now also U5.17 (I14); no longer U5.22 (I9)
- net at RVM1.2, SW_F1.9: now also U5.23 (I8); no longer U5.16 (I15)
Changed lines of the file:
@@
 	1150 4100 1550 4100
 Wire Wire Line
-	3350 4200 1650 4200
-Wire Wire Line
-	3400 4300 1750 4300
-Wire Wire Line
 	1150 4400 1850 4400
-Wire Wire Line
-	3500 4500 1950 4500
-Wire Wire Line
-	3550 4600 2050 4600
 Wire Wire Line
 	1150 4700 2700 4700
@@
 	2700 4700 2700 5300
 Wire Wire Line
-	3200 3050 3550 3050
-Wire Wire Line
-	3600 2350 3600 3050
-Wire Wire Line
-	3600 3050 3550 3050
-Wire Wire Line
-	3600 2350 8200 2350
-Wire Wire Line
-	3550 2950 3550 4600
-Wire Wire Line
-	3200 2350 3250 2350
-Wire Wire Line
-	3250 2350 3250 4000
-Wire Wire Line
-	3200 2450 3300 2450
-Wire Wire Line
-	3300 2450 3300 4100
-Wire Wire Line
-	3200 2550 3350 2550
-Wire Wire Line
-	3350 2550 3350 4200
-Wire Wire Line
-	3200 2650 3400 2650
-Wire Wire Line
-	3400 2650 3400 4300
-Wire Wire Line
-	3200 2750 3450 2750
-Wire Wire Line
-	3450 2750 3450 4400
-Wire Wire Line
-	3200 2850 3500 2850
-Wire Wire Line
-	3500 2850 3500 4500
-Wire Wire Line
-	3550 2950 3200 2950
+	3200 2450 3600 2450
 Wire Wire Line
 	1550 4100 1550 5200
 Wire Wire Line
 	1550 5200 1150 5200
-Connection ~ 1550 4100
-Wire Wire Line
-	1550 4100 3300 4100
 Wire Wire Line
 	1650 4200 1650 5300
 Wire Wire Line
 	1650 5300 1150 5300
-Connection ~ 1650 4200
-Wire Wire Line
-	1650 4200 1150 4200
 Wire Wire Line
 	1750 4300 1750 5400
 Wire Wire Line
 	1750 5400 1150 5400
-Connection ~ 1750 4300
 Wire Wire Line
 	1750 4300 1150 4300
@@
 Wire Wire Line
 	1150 5100 1450 5100
-Connection ~ 1450 4000
-Wire Wire Line
-	1450 4000 3250 4000
 Wire Wire Line
 	1850 4400 1850 5500
 Wire Wire Line
 	1850 5500 1150 5500
-Connection ~ 1850 4400
-Wire Wire Line
-	1850 4400 3450 4400
 Wire Wire Line
 	1950 4500 1950 5600
 Wire Wire Line
 	1950 5600 1150 5600
-Connection ~ 1950 4500
 Wire Wire Line
 	1950 4500 1150 4500
@@
 Wire Wire Line
 	2050 5700 1150 5700
+Wire Wire Line
+	2050 4600 1150 4600
+Wire Wire Line
+	3200 2350 8200 2350
+Wire Wire Line
+	3600 2450 3600 4600
+Wire Wire Line
+	3600 4600 2050 4600
 Connection ~ 2050 4600
 Wire Wire Line
-	2050 4600 1150 4600
-Text Label 1150 5100 2    50   ~ 0
+	1950 4500 3550 4500
+Wire Wire Line
+	3550 4500 3550 2550
+Connection ~ 1950 4500
+Wire Wire Line
+	3200 2550 3550 2550
+Wire Wire Line
+	3200 2650 3500 2650
+Wire Wire Line
+	3500 2650 3500 4400
+Wire Wire Line
+	3500 4400 1850 4400
+Connection ~ 1850 4400
+Wire Wire Line
+	1750 4300 3450 4300
+Wire Wire Line
+	3450 4300 3450 2750
+Wire Wire Line
+	3450 2750 3200 2750
+Connection ~ 1750 4300
+Wire Wire Line
+	3200 2850 3400 2850
+Wire Wire Line
+	3400 2850 3400 4200
+Wire Wire Line
+	1150 4200 1650 4200
+Connection ~ 1650 4200
+Wire Wire Line
+	1650 4200 3400 4200
+Connection ~ 1550 4100
+Wire Wire Line
+	3200 2950 3350 2950
+Wire Wire Line
+	1550 4100 3350 4100
+Wire Wire Line
+	3350 4100 3350 2950
+Connection ~ 1450 4000
+Wire Wire Line
+	3300 4000 3300 3050
+Wire Wire Line
+	3300 3050 3200 3050
+Wire Wire Line
+	1450 4000 3300 4000
+Text HLabel 1150 5100 0    50   Input ~ 0
 U5_8
-Text Label 1150 5200 2    50   ~ 0
+Text HLabel 1150 5200 0    50   Input ~ 0
 U5_9
-Text Label 1150 5300 2    50   ~ 0
+Text HLabel 1150 5300 0    50   Input ~ 0
 U5_10
-Text Label 1150 5400 2    50   ~ 0
+Text HLabel 1150 5400 0    50   Input ~ 0
 U5_11
-Text Label 1150 5500 2    50   ~ 0
+Text HLabel 1150 5500 0    50   Input ~ 0
 U5_12
-Text Label 1150 5600 2    50   ~ 0
+Text HLabel 1150 5600 0    50   Input ~ 0
 U5_13
-Text Label 1150 5700 2    50   ~ 0
+Text HLabel 1150 5700 0    50   Input ~ 0
 U5_14
 $EndSCHEMATC
