File: Clip Block Left.sch (KiCad schematic (older format))
At the start: 27 parts, among them J1 Conn_02x05_Odd_Even, SW1 B3F-5050, SW10 B3F-5050, SW11 B3F-5050, SW12 B3F-5050, SW13 B3F-5050, SW14 B3F-5050, SW15 B3F-5050, SW16 B3F-5050, SW2 B3F-5050, SW3 B3F-5050, SW4 B3F-5050, SW5 B3F-5050, SW6 B3F-5050, SW7 B3F-5050, SW8 B3F-5050, SW9 B3F-5050, U1 CD74HC4067M

Commit message: Updated Schematic and changed rotary pots
Better button symbol and flipped all rotary pots in the schematic so they've connected the right way round.

Changed the rotary pot footprints so the graphics match the ones I'm using.
Parts:
- SW1, SW10, SW11, SW12, SW13, SW14, SW15, SW16, SW2, SW3, SW4, SW5, SW6, SW7, SW8, SW9, SW_1, SW_2, SW_3, SW_4: symbol cp_midi_control_surface_002-rescue:SW_SPST_4_PIN-sw_spst_0 -> cunabulapress-symbols:SW_SPST_NO_Omron_B3F-5050
Changed lines of the file:
@@
 EESchema Schematic File Version 4
 LIBS:cp_midi_control_surface_002-cache
-EELAYER 30 0
+EELAYER 26 0
 EELAYER END
 $Descr A4 11693 8268
@@
 $EndDescr
 $Comp
-L cp_midi_control_surface_002-rescue:SW_SPST_4_PIN-sw_spst_0 SW?
+L cunabulapress-symbols:SW_SPST_NO_Omron_B3F-5050 SW?
 U 1 1 5C4BAAC6
 P 7500 2450
@@
 $EndComp
 $Comp
-L cp_midi_control_surface_002-rescue:SW_SPST_4_PIN-sw_spst_0 SW?
+L cunabulapress-symbols:SW_SPST_NO_Omron_B3F-5050 SW?
 U 1 1 5C4BAAC7
 P 7500 2850
@@
 $EndComp
 $Comp
-L cp_midi_control_surface_002-rescue:SW_SPST_4_PIN-sw_spst_0 SW?
+L cunabulapress-symbols:SW_SPST_NO_Omron_B3F-5050 SW?
 U 1 1 5C4BAAC8
 P 7500 3250
@@
 $EndComp
 $Comp
-L cp_midi_control_surface_002-rescue:SW_SPST_4_PIN-sw_spst_0 SW?
+L cunabulapress-symbols:SW_SPST_NO_Omron_B3F-5050 SW?
 U 1 1 5C4BAAC9
 P 7500 3650
@@
 $EndComp
 $Comp
-L cp_midi_control_surface_002-rescue:SW_SPST_4_PIN-sw_spst_0 SW?
+L cunabulapress-symbols:SW_SPST_NO_Omron_B3F-5050 SW?
 U 1 1 5C4B764F
 P 7500 4050
@@
 $EndComp
 $Comp
-L cp_midi_control_surface_002-rescue:SW_SPST_4_PIN-sw_spst_0 SW?
+L cunabulapress-symbols:SW_SPST_NO_Omron_B3F-5050 SW?
 U 1 1 5C4B8146
 P 7500 4450
@@
 $EndComp
 $Comp
-L cp_midi_control_surface_002-rescue:SW_SPST_4_PIN-sw_spst_0 SW?
+L cunabulapress-symbols:SW_SPST_NO_Omron_B3F-5050 SW?
 U 1 1 5C4B814C
 P 7500 4850
@@
 $EndComp
 $Comp
-L cp_midi_control_surface_002-rescue:SW_SPST_4_PIN-sw_spst_0 SW?
+L cunabulapress-symbols:SW_SPST_NO_Omron_B3F-5050 SW?
 U 1 1 5C4B8152
 P 7500 5250
@@
 $EndComp
 $Comp
-L cp_midi_control_surface_002-rescue:SW_SPST_4_PIN-sw_spst_0 SW?
+L cunabulapress-symbols:SW_SPST_NO_Omron_B3F-5050 SW?
 U 1 1 5C4B907B
 P 5100 2450
@@
 $EndComp
 $Comp
-L cp_midi_control_surface_002-rescue:SW_SPST_4_PIN-sw_spst_0 SW?
+L cunabulapress-symbols:SW_SPST_NO_Omron_B3F-5050 SW?
 U 1 1 5C4B9081
 P 5100 2850
@@
 $EndComp
 $Comp
-L cp_midi_control_surface_002-rescue:SW_SPST_4_PIN-sw_spst_0 SW?
+L cunabulapress-symbols:SW_SPST_NO_Omron_B3F-5050 SW?
 U 1 1 5C4B9087
 P 5100 3250
@@
 $EndComp
 $Comp
-L cp_midi_control_surface_002-rescue:SW_SPST_4_PIN-sw_spst_0 SW?
+L cunabulapress-symbols:SW_SPST_NO_Omron_B3F-5050 SW?
 U 1 1 5C4B908D
 P 5100 3650
@@
 $EndComp
 $Comp
-L cp_midi_control_surface_002-rescue:SW_SPST_4_PIN-sw_spst_0 SW?
+L cunabulapress-symbols:SW_SPST_NO_Omron_B3F-5050 SW?
 U 1 1 5C4B9093
 P 5100 4050
@@
 $EndComp
 $Comp
-L cp_midi_control_surface_002-rescue:SW_SPST_4_PIN-sw_spst_0 SW?
+L cunabulapress-symbols:SW_SPST_NO_Omron_B3F-5050 SW?
 U 1 1 5C4B9099
 P 5100 4450
@@
 $EndComp
 $Comp
-L cp_midi_control_surface_002-rescue:SW_SPST_4_PIN-sw_spst_0 SW?
+L cunabulapress-symbols:SW_SPST_NO_Omron_B3F-5050 SW?
 U 1 1 5C4B909F
 P 5100 4850
@@
 $EndComp
 $Comp
-L cp_midi_control_surface_002-rescue:SW_SPST_4_PIN-sw_spst_0 SW?
+L cunabulapress-symbols:SW_SPST_NO_Omron_B3F-5050 SW?
 U 1 1 5C4B90A5
 P 5100 5250
@@
 	5500 1150 7900 1150
 $Comp
-L cp_midi_control_surface_002-rescue:SW_SPST_4_PIN-sw_spst_0 SW_1
+L cunabulapress-symbols:SW_SPST_NO_Omron_B3F-5050 SW_1
 U 1 1 5D5A9C0C
 P 2100 3800
@@
 $EndComp
 $Comp
-L cp_midi_control_surface_002-rescue:SW_SPST_4_PIN-sw_spst_0 SW_2
+L cunabulapress-symbols:SW_SPST_NO_Omron_B3F-5050 SW_2
 U 1 1 5D5A9C13
 P 2100 4300
@@
 $EndComp
 $Comp
-L cp_midi_control_surface_002-rescue:SW_SPST_4_PIN-sw_spst_0 SW_3
+L cunabulapress-symbols:SW_SPST_NO_Omron_B3F-5050 SW_3
 U 1 1 5D5A9C1A
 P 2100 4800
@@
 $EndComp
 $Comp
-L cp_midi_control_surface_002-rescue:SW_SPST_4_PIN-sw_spst_0 SW_4
+L cunabulapress-symbols:SW_SPST_NO_Omron_B3F-5050 SW_4
 U 1 1 5D5A9C21
 P 2100 5300
