File: Clip Block Right.sch (KiCad schematic (older format))
At the start: 27 parts, among them J2 Conn_02x05_Odd_Even, SW17 B3F-5050, SW18 B3F-5050, SW19 B3F-5050, SW20 B3F-5050, SW21 B3F-5050, SW22 B3F-5050, SW23 B3F-5050, SW24 B3F-5050, SW25 B3F-5050, SW26 B3F-5050, SW27 B3F-5050, SW28 B3F-5050, SW29 B3F-5050, SW30 B3F-5050, SW31 B3F-5050, SW32 B3F-5050, U2 CD74HC4067M

Commit message: Updated Schematic and changed rotary pots
Better button symbol and flipped all rotary pots in the schematic so they've connected the right way round.

Changed the rotary pot footprints so the graphics match the ones I'm using.
Parts:
- SW17, SW18, SW19, SW20, SW21, SW22, SW23, SW24, SW25, SW26, SW27, SW28, SW29, SW30, SW31, SW32, SW_5, SW_6, SW_7, SW_8: symbol cp_midi_control_surface_002-rescue:SW_SPST_4_PIN-sw_spst_0 -> cunabulapress-symbols:SW_SPST_NO_Omron_B3F-5050
Changed lines of the file:
@@
 EESchema Schematic File Version 4
 LIBS:cp_midi_control_surface_002-cache
-EELAYER 30 0
+EELAYER 26 0
 EELAYER END
 $Descr A4 11693 8268
@@
 $EndDescr
 $Comp
-L cp_midi_control_surface_002-rescue:SW_SPST_4_PIN-sw_spst_0 SW?
+L cunabulapress-symbols:SW_SPST_NO_Omron_B3F-5050 SW?
 U 1 1 5C60BB62
 P 7500 2850
@@
 $EndComp
 $Comp
-L cp_midi_control_surface_002-rescue:SW_SPST_4_PIN-sw_spst_0 SW?
+L cunabulapress-symbols:SW_SPST_NO_Omron_B3F-5050 SW?
 U 1 1 5C60BB69
 P 7500 3250
@@
 $EndComp
 $Comp
-L cp_midi_control_surface_002-rescue:SW_SPST_4_PIN-sw_spst_0 SW?
+L cunabulapress-symbols:SW_SPST_NO_Omron_B3F-5050 SW?
 U 1 1 5C60BB70
 P 7500 3650
@@
 $EndComp
 $Comp
-L cp_midi_control_surface_002-rescue:SW_SPST_4_PIN-sw_spst_0 SW?
+L cunabulapress-symbols:SW_SPST_NO_Omron_B3F-5050 SW?
 U 1 1 5C60BB77
 P 7500 4050
@@
 $EndComp
 $Comp
-L cp_midi_control_surface_002-rescue:SW_SPST_4_PIN-sw_spst_0 SW?
+L cunabulapress-symbols:SW_SPST_NO_Omron_B3F-5050 SW?
 U 1 1 5C60BB7E
 P 7500 4450
@@
 $EndComp
 $Comp
-L cp_midi_control_surface_002-rescue:SW_SPST_4_PIN-sw_spst_0 SW?
+L cunabulapress-symbols:SW_SPST_NO_Omron_B3F-5050 SW?
 U 1 1 5C60BB8C
 P 7500 5250
@@
 $EndComp
 $Comp
-L cp_midi_control_surface_002-rescue:SW_SPST_4_PIN-sw_spst_0 SW?
+L cunabulapress-symbols:SW_SPST_NO_Omron_B3F-5050 SW?
 U 1 1 5C60BB93
 P 5100 2450
@@
 $EndComp
 $Comp
-L cp_midi_control_surface_002-rescue:SW_SPST_4_PIN-sw_spst_0 SW?
+L cunabulapress-symbols:SW_SPST_NO_Omron_B3F-5050 SW?
 U 1 1 5C60BB9A
 P 5100 2850
@@
 $EndComp
 $Comp
-L cp_midi_control_surface_002-rescue:SW_SPST_4_PIN-sw_spst_0 SW?
+L cunabulapress-symbols:SW_SPST_NO_Omron_B3F-5050 SW?
 U 1 1 5C60BBA8
 P 5100 3650
@@
 $EndComp
 $Comp
-L cp_midi_control_surface_002-rescue:SW_SPST_4_PIN-sw_spst_0 SW?
+L cunabulapress-symbols:SW_SPST_NO_Omron_B3F-5050 SW?
 U 1 1 5C60BBAF
 P 5100 4050
@@
 $EndComp
 $Comp
-L cp_midi_control_surface_002-rescue:SW_SPST_4_PIN-sw_spst_0 SW?
+L cunabulapress-symbols:SW_SPST_NO_Omron_B3F-5050 SW?
 U 1 1 5C60BBB6
 P 5100 4450
@@
 $EndComp
 $Comp
-L cp_midi_control_surface_002-rescue:SW_SPST_4_PIN-sw_spst_0 SW?
+L cunabulapress-symbols:SW_SPST_NO_Omron_B3F-5050 SW?
 U 1 1 5C60BBBD
 P 5100 4850
@@
 $EndComp
 $Comp
-L cp_midi_control_surface_002-rescue:SW_SPST_4_PIN-sw_spst_0 SW?
+L cunabulapress-symbols:SW_SPST_NO_Omron_B3F-5050 SW?
 U 1 1 5C60BBC4
 P 5100 5250
@@
 	2700 1150 2700 1250
 $Comp
-L cp_midi_control_surface_002-rescue:SW_SPST_4_PIN-sw_spst_0 SW?
+L cunabulapress-symbols:SW_SPST_NO_Omron_B3F-5050 SW?
 U 1 1 5C60BBA1
 P 5100 3250
@@
 NoConn ~ 7700 5250
 $Comp
-L cp_midi_control_surface_002-rescue:SW_SPST_4_PIN-sw_spst_0 SW?
+L cunabulapress-symbols:SW_SPST_NO_Omron_B3F-5050 SW?
 U 1 1 5C60BB5B
 P 7500 2450
@@
 NoConn ~ 7700 4950
 $Comp
-L cp_midi_control_surface_002-rescue:SW_SPST_4_PIN-sw_spst_0 SW?
+L cunabulapress-symbols:SW_SPST_NO_Omron_B3F-5050 SW?
 U 1 1 5C60BB85
 P 7500 4850
@@
 $EndComp
 $Comp
-L cp_midi_control_surface_002-rescue:SW_SPST_4_PIN-sw_spst_0 SW?
+L cunabulapress-symbols:SW_SPST_NO_Omron_B3F-5050 SW?
 U 1 1 5D610099
 P 2100 3800
@@
 $EndComp
 $Comp
-L cp_midi_control_surface_002-rescue:SW_SPST_4_PIN-sw_spst_0 SW?
+L cunabulapress-symbols:SW_SPST_NO_Omron_B3F-5050 SW?
 U 1 1 5D6100A0
 P 2100 4300
@@
 $EndComp
 $Comp
-L cp_midi_control_surface_002-rescue:SW_SPST_4_PIN-sw_spst_0 SW?
+L cunabulapress-symbols:SW_SPST_NO_Omron_B3F-5050 SW?
 U 1 1 5D6100A7
 P 2100 4800
@@
 $EndComp
 $Comp
-L cp_midi_control_surface_002-rescue:SW_SPST_4_PIN-sw_spst_0 SW?
+L cunabulapress-symbols:SW_SPST_NO_Omron_B3F-5050 SW?
 U 1 1 5D6100AE
 P 2100 5300
